Commit message: Jump base class

File: model/jump_2.urdf (robot description, URDF)
Before this commit: robot JumpRobot, 6 links, 5 joints
Joints:
- joint base: origin xyz=0 5 0 rpy=0 0 0 -> xyz=0 0 0 rpy=0 0 0
- joint base_r: axis 0 0 1 -> 1 0 0; limit effort=100 velocity=100 -> lower=-20 upper=20 effort=100 velocity=100; type continuous -> prismatic
